File: circuits/main/main.sch (KiCad schematic (older format))
At the start: 28 parts, among them J1 Port 1, J10 Adafruit_Ultimate_GPS, J2 Port 2, J3 Port 3, J4 Port 4, J5 VSELECT 1, J6 VSELECT 2, J7 VSELECT 3, J8 VSELECT 4, J9 Raspberry_Pi_2_3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

Commit message: f
Parts:
- 16MHz: symbol Device:Crystal -> main-rescue:Crystal-Device
- C1, C2, C3, C4, C5, C6: symbol Device:C_Small -> main-rescue:C_Small-Device
- R1, R3, R4, R5, R6, R7: symbol Device:R -> main-rescue:R-Device
- U1: symbol 74LVC244APW_112:74LVC244APW,112 -> main-rescue:74LVC244APW,112-74LVC244APW_112
Changed lines of the file:
@@
 $EndDescr
 $Comp
-L Device:R R4
+L main-rescue:R-Device R4
 U 1 1 5A51638A
 P 1250 1050
@@
 $EndComp
 $Comp
-L Device:R R5
+L main-rescue:R-Device R5
 U 1 1 5A5164FF
 P 1500 1050
@@
 $EndComp
 $Comp
-L Device:R R6
+L main-rescue:R-Device R6
 U 1 1 5A516CD7
 P 2500 1050
@@
 $EndComp
 $Comp
-L Device:R R7
+L main-rescue:R-Device R7
 U 1 1 5A516D34
 P 2750 1050
@@
 $EndComp
 $Comp
-L power:+3.3V #PWR?
+L main-rescue:+3.3V-power #PWR?
 U 1 1 5A5170AD
 P 1250 800
@@
 $EndComp
 $Comp
-L power:+5V #PWR?
+L main-rescue:+5V-power #PWR?
 U 1 1 5A517131
 P 2750 800
@@
 3.3V_SCL
 $Comp
-L power:+5V #PWR?
+L main-rescue:+5V-power #PWR?
 U 1 1 5A51829A
 P 5000 800
@@
 $EndComp
 $Comp
-L power:GND #PWR?
+L main-rescue:GND-power #PWR?
 U 1 1 5A5183B1
 P 5000 3600
@@
 Pi_CE0
 $Comp
-L power:GND #PWR?
+L main-rescue:GND-power #PWR?
 U 1 1 5A51AFDC
 P 7050 1600
@@
 $EndComp
 $Comp
-L power:+3.3V #PWR?
+L main-rescue:+3.3V-power #PWR?
 U 1 1 5A51B010
 P 7050 800
@@
 $EndComp
 $Comp
-L power:+3.3V #PWR?
+L main-rescue:+3.3V-power #PWR?
 U 1 1 5A51C3A8
 P 2200 2400
@@
 $EndComp
 $Comp
-L power:+5V #PWR?
+L main-rescue:+5V-power #PWR?
 U 1 1 5A51C3EC
 P 1950 2400
@@
 $EndComp
 $Comp
-L power:GND #PWR?
+L main-rescue:GND-power #PWR?
 U 1 1 5A51C430
 P 2200 3100
@@
 $EndComp
 $Comp
-L power:+5VP #PWR?
+L main-rescue:+5VP-power #PWR?
 U 1 1 5A51D86B
 P 1400 2700
@@
 $EndComp
 $Comp
-L power:+3.3V #PWR?
+L main-rescue:+3.3V-power #PWR?
 U 1 1 5A51E05A
 P 2200 3500
@@
 $EndComp
 $Comp
-L power:+5V #PWR?
+L main-rescue:+5V-power #PWR?
 U 1 1 5A51E0A2
 P 2000 3500
@@
 $EndComp
 $Comp
-L power:GND #PWR?
+L main-rescue:GND-power #PWR?
 U 1 1 5A51E145
 P 2200 4200
@@
 $EndComp
 $Comp
-L power:+3.3V #PWR?
+L main-rescue:+3.3V-power #PWR?
 U 1 1 5A51E1C1
 P 2200 4600
@@
 $EndComp
 $Comp
-L power:+5V #PWR?
+L main-rescue:+5V-power #PWR?
 U 1 1 5A51E257
 P 2000 4600
@@
 $EndComp
 $Comp
-L power:GND #PWR?
+L main-rescue:GND-power #PWR?
 U 1 1 5A51E362
 P 2200 5300
@@
 $EndComp
 $Comp
-L power:+3.3V #PWR?
+L main-rescue:+3.3V-power #PWR?
 U 1 1 5A51E3AA
 P 2200 5700
@@
 $EndComp
 $Comp
-L power:+5V #PWR?
+L main-rescue:+5V-power #PWR?
 U 1 1 5A51E3F2
 P 2000 5700
@@
 $EndComp
 $Comp
-L power:GND #PWR?
+L main-rescue:GND-power #PWR?
 U 1 1 5A51E6BA
 P 2200 6400
@@
 $EndComp
 $Comp
-L power:+5V #PWR?
+L main-rescue:+5V-power #PWR?
 U 1 1 5A826BFE
 P 1600 2700
@@
 $EndComp
 $Comp
-L power:+5VP #PWR?
+L main-rescue:+5VP-power #PWR?
 U 1 1 5A826CCB
 P 1400 3800
@@
 $EndComp
 $Comp
-L power:+5V #PWR?
+L main-rescue:+5V-power #PWR?
 U 1 1 5A826CD7
 P 1600 3800
@@
 $EndComp
 $Comp
-L power:+5VP #PWR?
+L main-rescue:+5VP-power #PWR?
 U 1 1 5A826DB5
 P 1400 4900
@@
 $EndComp
 $Comp
-L power:+5V #PWR?
+L main-rescue:+5V-power #PWR?
 U 1 1 5A826DC1
 P 1600 4900
@@
 $EndComp
 $Comp
-L power:+5VP #PWR?
+L main-rescue:+5VP-power #PWR?
 U 1 1 5A826EEE
 P 1400 6000
@@
 $EndComp
 $Comp
-L power:+5V #PWR?
+L main-rescue:+5V-power #PWR?
 U 1 1 5A826EFA
 P 1600 6000
@@
 AVR_RST
 $Comp
-L Device:R R3
+L main-rescue:R-Device R3
 U 1 1 5A8291E8
 P 6850 5700
@@
 $EndComp
 $Comp
-L power:+5VP #PWR?
+L main-rescue:+5VP-power #PWR?
 U 1 1 5A829FCD
 P 7200 5600
@@
 AVR_D4
 $Comp
-L Device:C_Small C3
+L main-rescue:C_Small-Device C3
 U 1 1 5A82A4ED
 P 3800 4250
@@
 $EndComp
 $Comp
-L power:+5VP #PWR?
+L main-rescue:+5VP-power #PWR?
 U 1 1 5A82A947
 P 4000 4150
@@
 $EndComp
 $Comp
-L Device:C_Small C4
+L main-rescue:C_Small-Device C4
 U 1 1 5A82AA5F
 P 3800 4550
@@
 $EndComp
 $Comp
-L power:GND #PWR?
+L main-rescue:GND-power #PWR?
 U 1 1 5A82ADF7
 P 3600 5300
@@
 $EndComp
 $Comp
-L power:GND #PWR?
+L main-rescue:GND-power #PWR?
 U 1 1 5A82AFC9
 P 4000 6600
@@
 AVR_D7
 $Comp
-L Device:Crystal 16MHz
+L main-rescue:Crystal-Device 16MHz
 U 1 1 5A9B414C
 P 6800 4900
@@
 $EndComp
 $Comp
-L Device:C_Small C1
+L main-rescue:C_Small-Device C1
 U 1 1 5A9B4351
 P 7100 5100
@@
 $EndComp
 $Comp
-L Device:C_Small C2
+L main-rescue:C_Small-Device C2
 U 1 1 5A9B4456
 P 7100 4700
@@
 $EndComp
 $Comp
-L power:GND #PWR?
+L main-rescue:GND-power #PWR?
 U 1 1 5A9B4E12
 P 7400 5200
@@
 ADC7
 $Comp
-L Device:C_Small C5
+L main-rescue:C_Small-Device C5
 U 1 1 5C427D88
 P 3800 4850
@@
 	4000 6550 4000 6600
 $Comp
-L Device:C_Small C6
+L main-rescue:C_Small-Device C6
 U 1 1 5C49CBB5
 P 3800 5150
@@
 	6600 5700 6000 5700
 $Comp
-L 74LVC244APW_112:74LVC244APW,112 U1
+L main-rescue:74LVC244APW,112-74LVC244APW_112 U1
 U 1 1 5C2C23F0
 P 9400 4800
@@
 Pi_CE0
 $Comp
-L power:+3.3V #PWR?
+L main-rescue:+3.3V-power #PWR?
 U 1 1 5C2C3A64
 P 8100 4200
@@
 $EndComp
 $Comp
-L Device:R R1
+L main-rescue:R-Device R1
 U 1 1 5C2D35AA
 P 8350 4300
@@
 $EndComp
 $Comp
-L power:GND #PWR?
+L main-rescue:GND-power #PWR?
 U 1 1 5C2D3BEC
 P 8600 5800
@@
 	8600 5700 8600 5800
 $Comp
-L power:+3.3V #PWR?
+L main-rescue:+3.3V-power #PWR?
 U 1 1 5C33B0D4
 P 8600 4100
@@
 ATMEGA Programmer
 $Comp
-L power:GND #PWR?
+L main-rescue:GND-power #PWR?
 U 1 1 5E497E40
 P 8650 1300
@@
 $EndComp
 $Comp
-L power:+5VP #PWR?
+L main-rescue:+5VP-power #PWR?
 U 1 1 5E4A241A
 P 8200 1150
